Commit message: 衝突形状を簡略化し、実時間係数を 0.26 から 1.00 に戻す
jetbot_real.urdf.xacro は 20 個すべてのリンクで視覚用の高精細 STL を
そのまま衝突形状にも使っていた。DART が毎ステップこれを衝突判定するため、
ロボットを spawn した時点で実時間係数が 1.0 から 0.26 に落ちていた。

  collision の三角形 合計 745,410
    nano_link         374,540
    imu_link          100,902
    base_scan          79,672
    camera_link        56,300
    caster_*_link      23,258 x 2
    wheel_*_tire       13,324 x 2

## 置き換えの方針

各 STL の頂点境界ボックスを実測し、接地するかどうかで扱いを分けた。

| 対象 | 置き換え | 根拠 |
|------|----------|------|
| wheel_*_tire | 円柱 r=0.0325 l=0.029 | AABB 0.0650x0.0650x0.0290。DiffDrive の wheel_radius 0.033 と整合。関節の rpy=-pi/2 (x 軸) によりリンク座標系の z が車軸なので円柱の既定軸と一致する |
| caster_*_link | 球 r=0.019 | AABB の y 方向 0.0380 の半分。接地点が元メッシュと一致する位置に置いた |
| wheel_*_link, wheel_*_rim | 衝突形状を削除 | タイヤの内側で接地しない |
| 他 12 リンク | 各自の AABB から箱 | 固定関節で base_link にまとめられ接地しない |

単一の大きな箱にまとめるとアンテナ (高さ 0.126) やカメラ (前方 0.115) まで
覆って実機より太るため、リンクごとの箱にした。1 個 12 三角形なので合計でも
約 600 三角形に収まる。

視覚形状 (<visual>) は無改変。リンク名・関節名・慣性も変更していないので
DiffDrive の left_joint / right_joint 指定や TF 構成に影響しない。

## 実時間係数の実測

| 条件 | RTF |
|------|-----|
| 変更前 (高精細メッシュ) + bridge | 0.0094 |
| 変更後 + bridge にセンサ含む | 0.0025 |
| 変更後 + bridge_sensors:=false | 1.000 |
| 変更後 + gz 単体 (bridge なし) | 1.000 |

## 以前の報告を訂正する

コミット 15c4fb4 で「Sensors システムは原因ではない」「ブリッジの購読では
ない」と書いたが、これは誤りだった。当時は衝突形状のコストが支配的で
(0.26)、センサ描画のコストが埋もれて見えなかった。

衝突形状を直した今、bridge_sensors の有無で 400 倍の差が出る。
ros_gz_bridge が /image_raw2 と /scan を購読すると Sensors システムが描画を
始め、GPU が使えない環境では 640x480 カメラ 30 Hz と 1147 点 LiDAR を CPU で
描くことになる。launch の docstring を実測値に基づく記述へ差し替えた。

## 走行の検証

bridge_sensors:=false (RTF 1.000) で cmd_vel に 0.3 m/s を 6 秒送り、
odom の移動距離が 1.450 m になることを確認した。理論値 1.8 m に対し、
_action_to_cmd の accel_rate による立ち上がりと publish 開始の遅れを
含めて妥当な値である。

Refs #5

Co-Authored-By: Claude Opus 5 <noreply@anthropic.com>

File: jetbot_world/urdf/jetbot_real.urdf.xacro (robot description, xacro)
@@ -32,8 +32,11 @@
       </material>
     </visual>
-    <collision>
-      <origin rpy="0 0 0" xyz="0 0 0"/>
-      <geometry>
-        <mesh filename="package://jetbot_world/meshes/other_parts/base_link.STL"/>
+    <!-- 高精細メッシュ (3156 三角形) を境界ボックスの箱で
+         近似した。固定関節で base_link にまとめられるリンクで、
+         接地しないため形状の細部は挙動に影響しない。 -->
+    <collision>
+      <origin rpy="0 0 0" xyz="0.000000 0.000000 0.005922"/>
+      <geometry>
+        <box size="0.199396 0.184447 0.093266"/>
       </geometry>
     </collision>
@@ -54,10 +57,6 @@
       </material>
     </visual>
-    <collision>
-      <origin rpy="0 0 0" xyz="0 0 0"/>
-      <geometry>
-        <mesh filename="package://jetbot_world/meshes/wheels/wheel_right_link.STL"/>
-      </geometry>
-    </collision>
+    <!-- 衝突形状を削除した。タイヤの内側にあり接地しない。
+         元は meshes/wheels/wheel_right_link.STL (1002 三角形) を使っていた。 -->
   </link>
   <joint name="wheel_right_joint" type="continuous">
@@ -90,10 +89,6 @@
       </material>
     </visual>
-    <collision>
-      <origin rpy="0 0 0" xyz="0 0 0"/>
-      <geometry>
-        <mesh filename="package://jetbot_world/meshes/wheels/wheel_right_rim.STL"/>
-      </geometry>
-    </collision>
+    <!-- 衝突形状を削除した。タイヤの内側にあり接地しない。
+         元は meshes/wheels/wheel_right_rim.STL (3284 三角形) を使っていた。 -->
   </link>
   <joint name="wheel_right_rim_joint" type="fixed">
@@ -118,8 +113,11 @@
       </material>
     </visual>
-    <collision>
-      <origin rpy="0 0 0" xyz="0 0 0"/>
-      <geometry>
-        <mesh filename="package://jetbot_world/meshes/wheels/wheel_right_tire.STL"/>
+    <!-- 接地するリンク。高精細メッシュ (13324 三角形) を
+         円柱 r=0.0325 l=0.029 で近似した。寸法は元メッシュの境界ボックス
+         (0.0650, 0.0650, 0.0290) から決めている。 -->
+    <collision>
+      <origin rpy="0 0 0" xyz="0.000008 0.000421 0.000200"/>
+      <geometry>
+        <cylinder radius="0.0325" length="0.029"/>
       </geometry>
     </collision>
@@ -146,10 +144,6 @@
       </material>
     </visual>
-    <collision>
-      <origin rpy="0 0 0" xyz="0 0 0"/>
-      <geometry>
-        <mesh filename="package://jetbot_world/meshes/wheels/wheel_left_link.STL"/>
-      </geometry>
-    </collision>
+    <!-- 衝突形状を削除した。タイヤの内側にあり接地しない。
+         元は meshes/wheels/wheel_left_link.STL (1002 三角形) を使っていた。 -->
   </link>
   <joint name="wheel_left_joint" type="continuous">
@@ -176,10 +170,6 @@
       </material>
     </visual>
-    <collision>
-      <origin rpy="0 0 0" xyz="0 0 0"/>
-      <geometry>
-        <mesh filename="package://jetbot_world/meshes/wheels/wheel_left_rim.STL"/>
-      </geometry>
-    </collision>
+    <!-- 衝突形状を削除した。タイヤの内側にあり接地しない。
+         元は meshes/wheels/wheel_left_rim.STL (3284 三角形) を使っていた。 -->
   </link>
   <joint name="wheel_left_rim_joint" type="fixed">
@@ -204,8 +194,11 @@
       </material>
     </visual>
-    <collision>
-      <origin rpy="0 0 0" xyz="0 0 0"/>
-      <geometry>
-        <mesh filename="package://jetbot_world/meshes/wheels/wheel_left_tire.STL"/>
+    <!-- 接地するリンク。高精細メッシュ (13324 三角形) を
+         円柱 r=0.0325 l=0.029 で近似した。寸法は元メッシュの境界ボックス
+         (0.0650, 0.0650, 0.0290) から決めている。 -->
+    <collision>
+      <origin rpy="0 0 0" xyz="0.000417 -0.000058 -0.000200"/>
+      <geometry>
+        <cylinder radius="0.0325" length="0.029"/>
       </geometry>
     </collision>
@@ -232,8 +225,11 @@
       </material>
     </visual>
-    <collision>
-      <origin rpy="0 0 0" xyz="0 0 0"/>
-      <geometry>
-        <mesh filename="package://jetbot_world/meshes/realsense/camera_mount_link.STL"/>
+    <!-- 高精細メッシュ (276 三角形) を境界ボックスの箱で
+         近似した。固定関節で base_link にまとめられるリンクで、
+         接地しないため形状の細部は挙動に影響しない。 -->
+    <collision>
+      <origin rpy="0 0 0" xyz="0.089169 -0.000050 0.047555"/>
+      <geometry>
+        <box size="0.011738 0.061000 0.012000"/>
       </geometry>
     </collision>
@@ -260,8 +256,11 @@
       </material>
     </visual>
-    <collision>
-      <origin rpy="0 0 0" xyz="0 0 0"/>
-      <geometry>
-        <mesh filename="package://jetbot_world/meshes/realsense/camera_link.STL"/>
+    <!-- 高精細メッシュ (56300 三角形) を境界ボックスの箱で
+         近似した。固定関節で base_link にまとめられるリンクで、
+         接地しないため形状の細部は挙動に影響しない。 -->
+    <collision>
+      <origin rpy="0 0 0" xyz="0.105063 0.000030 0.047555"/>
+      <geometry>
+        <box size="0.020050 0.098840 0.023000"/>
       </geometry>
     </collision>
@@ -288,8 +287,11 @@
       </material>
     </visual>
-    <collision>
-      <origin rpy="0 0 0" xyz="0 0 0"/>
-      <geometry>
-        <mesh filename="package://jetbot_world/meshes/other_parts/caster_back_link.STL"/>
+    <!-- 接地するリンク。高精細メッシュ (23258 三角形) を
+         球 r=0.019 で近似した。寸法は元メッシュの境界ボックス
+         (0.0455, 0.0380, 0.0400) から決めている。 -->
+    <collision>
+      <origin rpy="0 0 0" xyz="-0.005748 0.017682 0.000000"/>
+      <geometry>
+        <sphere radius="0.019"/>
       </geometry>
     </collision>
@@ -316,8 +318,11 @@
       </material>
     </visual>
-    <collision>
-      <origin rpy="0 0 0" xyz="0 0 0"/>
-      <geometry>
-        <mesh filename="package://jetbot_world/meshes/other_parts/caster_front_link.STL"/>
+    <!-- 接地するリンク。高精細メッシュ (23258 三角形) を
+         球 r=0.019 で近似した。寸法は元メッシュの境界ボックス
+         (0.0455, 0.0380, 0.0400) から決めている。 -->
+    <collision>
+      <origin rpy="0 0 0" xyz="-0.005748 0.015300 0.000000"/>
+      <geometry>
+        <sphere radius="0.019"/>
       </geometry>
     </collision>
@@ -344,8 +349,11 @@
       </material>
     </visual>
-    <collision>
-      <origin rpy="0 0 0" xyz="0 0 0"/>
-      <geometry>
-        <mesh filename="package://jetbot_world/meshes/other_parts/imu_link.STL"/>
+    <!-- 高精細メッシュ (100902 三角形) を境界ボックスの箱で
+         近似した。固定関節で base_link にまとめられるリンクで、
+         接地しないため形状の細部は挙動に影響しない。 -->
+    <collision>
+      <origin rpy="0 0 0" xyz="-0.002854 -0.000460 -0.008186"/>
+      <geometry>
+        <box size="0.137467 0.108247 0.030150"/>
       </geometry>
     </collision>
@@ -372,8 +380,11 @@
       </material>
     </visual>
-    <collision>
-      <origin rpy="0 0 0" xyz="0 0 0"/>
-      <geometry>
-        <mesh filename="package://jetbot_world/meshes/other_parts/base_scan.STL"/>
+    <!-- 高精細メッシュ (79672 三角形) を境界ボックスの箱で
+         近似した。固定関節で base_link にまとめられるリンクで、
+         接地しないため形状の細部は挙動に影響しない。 -->
+    <collision>
+      <origin rpy="0 0 0" xyz="-0.012854 0.000000 -0.000300"/>
+      <geometry>
+        <box size="0.097488 0.071776 0.051400"/>
       </geometry>
     </collision>
@@ -400,8 +411,11 @@
       </material>
     </visual>
-    <collision>
-      <origin rpy="0 0 0" xyz="0 0 0"/>
-      <geometry>
-        <mesh filename="package://jetbot_world/meshes/other_parts/left_motor_link.STL"/>
+    <!-- 高精細メッシュ (8618 三角形) を境界ボックスの箱で
+         近似した。固定関節で base_link にまとめられるリンクで、
+         接地しないため形状の細部は挙動に影響しない。 -->
+    <collision>
+      <origin rpy="0 0 0" xyz="0.000763 0.043300 -0.022000"/>
+      <geometry>
+        <box size="0.038526 0.072600 0.036967"/>
       </geometry>
     </collision>
@@ -428,8 +442,11 @@
       </material>
     </visual>
-    <collision>
-      <origin rpy="0 0 0" xyz="0 0 0"/>
-      <geometry>
-        <mesh filename="package://jetbot_world/meshes/other_parts/right_motor_link.STL"/>
+    <!-- 高精細メッシュ (8618 三角形) を境界ボックスの箱で
+         近似した。固定関節で base_link にまとめられるリンクで、
+         接地しないため形状の細部は挙動に影響しない。 -->
+    <collision>
+      <origin rpy="0 0 0" xyz="-0.000763 -0.043300 -0.022000"/>
+      <geometry>
+        <box size="0.038526 0.072600 0.036967"/>
       </geometry>
     </collision>
@@ -456,8 +473,11 @@
       </material>
     </visual>
-    <collision>
-      <origin rpy="0 0 0" xyz="0 0 0"/>
-      <geometry>
-        <mesh filename="package://jetbot_world/meshes/other_parts/upper_plate_link.STL"/>
+    <!-- 高精細メッシュ (680 三角形) を境界ボックスの箱で
+         近似した。固定関節で base_link にまとめられるリンクで、
+         接地しないため形状の細部は挙動に影響しない。 -->
+    <collision>
+      <origin rpy="0 0 0" xyz="-0.006950 0.000300 0.062186"/>
+      <geometry>
+        <box size="0.100000 0.079000 0.003000"/>
       </geometry>
     </collision>
@@ -484,8 +504,11 @@
       </material>
     </visual>
-    <collision>
-      <origin rpy="0 0 0" xyz="0 0 0"/>
-      <geometry>
-        <mesh filename="package://jetbot_world/meshes/other_parts/antenna_link.STL"/>
+    <!-- 高精細メッシュ (28672 三角形) を境界ボックスの箱で
+         近似した。固定関節で base_link にまとめられるリンクで、
+         接地しないため形状の細部は挙動に影響しない。 -->
+    <collision>
+      <origin rpy="0 0 0" xyz="-0.066000 0.000000 0.047300"/>
+      <geometry>
+        <box size="0.009980 0.130000 0.125700"/>
       </geometry>
     </collision>
@@ -512,8 +535,11 @@
       </material>
     </visual>
-    <collision>
-      <origin rpy="0 0 0" xyz="0 0 0"/>
-      <geometry>
-        <mesh filename="package://jetbot_world/meshes/other_parts/bolt1_link.STL"/>
+    <!-- 高精細メッシュ (1888 三角形) を境界ボックスの箱で
+         近似した。固定関節で base_link にまとめられるリンクで、
+         接地しないため形状の細部は挙動に影響しない。 -->
+    <collision>
+      <origin rpy="0 0 0" xyz="0.000000 0.000000 0.025843"/>
+      <geometry>
+        <box size="0.172680 0.095404 0.069686"/>
       </geometry>
     </collision>
@@ -540,8 +566,11 @@
       </material>
     </visual>
-    <collision>
-      <origin rpy="0 0 0" xyz="0 0 0"/>
-      <geometry>
-        <mesh filename="package://jetbot_world/meshes/other_parts/bolt2_link.STL"/>
+    <!-- 高精細メッシュ (352 三角形) を境界ボックスの箱で
+         近似した。固定関節で base_link にまとめられるリンクで、
+         接地しないため形状の細部は挙動に影響しない。 -->
+    <collision>
+      <origin rpy="0 0 0" xyz="-0.001950 0.000300 0.076186"/>
+      <geometry>
+        <box size="0.074650 0.061369 0.025000"/>
       </geometry>
     </collision>
@@ -568,8 +597,11 @@
       </material>
     </visual>
-    <collision>
-      <origin rpy="0 0 0" xyz="0 0 0"/>
-      <geometry>
-        <mesh filename="package://jetbot_world/meshes/other_parts/nano_link.STL"/>
+    <!-- 高精細メッシュ (374540 三角形) を境界ボックスの箱で
+         近似した。固定関節で base_link にまとめられるリンクで、
+         接地しないため形状の細部は挙動に影響しない。 -->
+    <collision>
+      <origin rpy="0 0 0" xyz="-0.006950 0.001313 0.048048"/>
+      <geometry>
+        <box size="0.100000 0.081025 0.042290"/>
       </geometry>
     </collision>
